File: KiCad/gamepad.kicad_pcb (KiCad board)
At the start: 2 copper layers, 0 parts

Commit message: feat: gamepad cad and kicad done and printable
Parts:
- added C2: 10u, Capacitor_Tantalum_SMD:CP_EIA-1608-10_AVX-L_HandSolder, F.Cu at (84.9, 27.5)
- added C3: 10u, Capacitor_Tantalum_SMD:CP_EIA-1608-10_AVX-L_HandSolder, F.Cu at (78.9, 27.7)
- added C4: 100n, Capacitor_Tantalum_SMD:CP_EIA-1608-10_AVX-L_HandSolder, F.Cu at (69.2, 32.5)
- added J2: USB_C_Receptacle_USB2.0_16P, Connector_USB:USB_C_Receptacle_HRO_TYPE-C-31-M-12, F.Cu at (71.9, 16.1)
- added J4: Flash_Pin, Connector_PinHeader_2.54mm:PinHeader_1x03_P2.54mm_Vertical, F.Cu at (81.8, 46.6)
- added J5: UART, Connector_PinHeader_2.54mm:PinHeader_1x02_P2.54mm_Vertical, F.Cu at (80.4, 37.0)
- added R1: 5.1K, Resistor_SMD:R_0805_2012Metric_Pad1.20x1.40mm_HandSolder, F.Cu at (63.6, 21.6)
- added R10: 10K, Resistor_SMD:R_0805_2012Metric_Pad1.20x1.40mm_HandSolder, F.Cu at (111.0, 46.0)
- added R11: 10K, Resistor_SMD:R_0805_2012Metric_Pad1.20x1.40mm_HandSolder, F.Cu at (84.3, 20.9)
- added R12: 10K, Resistor_SMD:R_0805_2012Metric_Pad1.20x1.40mm_HandSolder, F.Cu at (57.2, 26.7)
- added R13: 10K, Resistor_SMD:R_0805_2012Metric_Pad1.20x1.40mm_HandSolder, F.Cu at (63.0, 50.9)
- added R14: 10K, Resistor_SMD:R_0805_2012Metric_Pad1.20x1.40mm_HandSolder, F.Cu at (53.5, 52.4)
- added R2: 5.1K, Resistor_SMD:R_0805_2012Metric_Pad1.20x1.40mm_HandSolder, F.Cu at (79.3, 19.3)
- added R3: 1K, Resistor_SMD:R_0805_2012Metric_Pad1.20x1.40mm_HandSolder, F.Cu at (82.8, 42.9)
- added R4: 1K5, Resistor_SMD:R_0805_2012Metric_Pad1.20x1.40mm_HandSolder, F.Cu at (73.8, 26.1)
- added R5: 47, Resistor_SMD:R_0805_2012Metric_Pad1.20x1.40mm_HandSolder, F.Cu at (73.2, 29.1)
- added R6: 47, Resistor_SMD:R_0805_2012Metric_Pad1.20x1.40mm_HandSolder, F.Cu at (71.1, 29.1)
- added R7: 10K, Resistor_SMD:R_0805_2012Metric_Pad1.20x1.40mm_HandSolder, F.Cu at (92.2, 28.0)
- added R8: 10K, Resistor_SMD:R_0805_2012Metric_Pad1.20x1.40mm_HandSolder, F.Cu at (89.2, 42.0)
- added R9: 10K, Resistor_SMD:R_0805_2012Metric_Pad1.20x1.40mm_HandSolder, F.Cu at (92.7, 52.5)
- added SW1: X, Button_Switch_THT:SW_PUSH_6mm, F.Cu at (99.7, 23.1)
- added SW2: Y, Button_Switch_THT:SW_PUSH_6mm, F.Cu at (89.1, 33.6)
- added SW3: A, Button_Switch_THT:SW_PUSH_6mm, F.Cu at (99.6, 44.2)
- added SW4: B, Button_Switch_THT:SW_PUSH_6mm, F.Cu at (115.7, 32.6)
- added SW5: SR, Connector_Wire:SolderWire-0.5sqmm_1x02_P4.6mm_D0.9mm_OD2.1mm, F.Cu at (94.9, 21.0)
- added SW6: SL, Connector_Wire:SolderWire-0.5sqmm_1x02_P4.6mm_D0.9mm_OD2.1mm, F.Cu at (48.9, 21.0)
- added SW7: Start, Button_Switch_THT:SW_PUSH_6mm, F.Cu at (68.7, 45.7)
- added U1: XC6206PxxxMR, Package_TO_SOT_SMD:SOT-23-3, F.Cu at (81.9, 27.6)
- added U2: CH32V003FxPx, Package_SO:TSSOP-20_4.4x6.5mm_P0.65mm, F.Cu at (71.5, 37.6)
- added U3: COM-09032, COM-09032:XDCR_COM-09032, F.Cu at (39.7, 37.8)
Routing:
- net VDD: track 0.00 -> 302.3 mm, vias 0 -> 5
- net Button_B: track 0.00 -> 101.2 mm, vias 0 -> 1
- net Button_A: track 0.00 -> 76.7 mm, vias 0 -> 1
- net GND: track 0.00 -> 74.8 mm, vias 0 -> 7
- net Analog_X: track 0.00 -> 45.1 mm, vias 0 -> 1
- net Analog_SW: track 0.00 -> 36.8 mm, vias 0 -> 1
- net Button_X: track 0.00 -> 35.2 mm, vias 0 -> 1
- net Button_Y: track 0.00 -> 30.9 mm, vias 0 -> 1
- net +5V: track 0.00 -> 30.8 mm, vias 0 -> 2
- net Button_SR: track 0.00 -> 30.4 mm, vias 0 -> 1
- net Button_Start: track 0.00 -> 29.5 mm, vias 0 -> 1
- net Button_SL: track 0.00 -> 23.6 mm, vias 0 -> 1
- net Analog_Y: track 0.00 -> 23.2 mm, vias 0 -> 1
- net D-: track 0.00 -> 15.5 mm
- net D+: track 0.00 -> 15.2 mm, vias 0 -> 2
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- added copper zone on B.Cu, net GND
- added copper zone on F.Cu, net GND
Other:
- board outline added: 104.9 x 49.4 mm
