File: KiCad/gamepad.kicad_sch (KiCad schematic)
At the start: 31 parts, among them J2 USB_C_Receptacle_USB2.0_16P, J4 Flash_Pin, J5 UART, SW1 X, SW2 Y, SW3 A, SW4 B, SW5 SR, SW6 SL, SW7 SL, U1 XC6206PxxxMR, U2 CH32V003FxPx, U3 COM-09032

Commit message: feat: gamepad cad and kicad done and printable
Parts:
- removed R4: 10K, Resistor_SMD:R_0805_2012Metric_Pad1.20x1.40mm_HandSolder, symbol Device:R
- SW1, SW2, SW3, SW4: footprint (none) -> Button_Switch_THT:SW_PUSH_6mm
- SW5, SW6: footprint (none) -> Connector_Wire:SolderWire-0.5sqmm_1x02_P4.6mm_D0.9mm_OD2.1mm
- SW7: value SL -> Start; footprint (none) -> Button_Switch_THT:SW_PUSH_6mm
- renumbered R11 to R10, R12 to R11, R13 to R12, R14 to R13, R15 to R14, R5 to R4, R6 to R5, R7 to R6, R8 to R7, R9 to R8, R10 to R9
Connections:
- net FLS_VDD is gone; now on net VDD: J4.2 (Pin_2), R3.2
- net Analog_X: now also U2.19 (PD2); no longer U2.14 (PC4)
- net Analog_Y: now also U2.14 (PC4); no longer U2.1 (PD4)
- net Button_A: now also U2.16 (PC6); no longer U2.17 (PC7)
- net Button_B: now also U2.15 (PC5); no longer U2.16 (PC6)
- net Button_SL: now also U2.10 (PC0); no longer U2.11 (PC1)
- net Button_SR: now also U2.4 (PD7); no longer U2.13 (PC3)
- net Button_Start: now also U2.17 (PC7); no longer U2.15 (PC5)
- net Button_X: now also U2.1 (PD4); no longer U2.19 (PD2)
- no-connect marks 4 -> 5
